Commit message: Load testing in Gazebo, redesign decision in changelog
- tools/torque_monitor.py: live joint torque vs each joint's servo
  (OK / HOT / FAIL), MG996R on shoulder_lift, elbow_flex, wrist_flex.
- Gazebo payload_kg:= launch option: test mass at the gripper (Gazebo only).
- ava.urdf regenerated from the current xacro.
- CHANGELOG: SO-101 failed the load test (weight at the end of the arm);
  switching to an open model built for 2x MG996R + 4x SG90, redraw in progress.
- dashboard: part measuring, Automatic-mode confirmation.

Co-Authored-By: Claude Opus 5.5 <noreply@anthropic.com>

File: ros2_ws/src/ava_description/urdf/ava.urdf (robot description, URDF)
Before this commit: robot ava, 9 links, 8 joints
Links:
- added link wrist_camera_body_link, mass 0.015; collision mesh filename=package://ava_description/meshes/wrist_camera_so101_v1.stl; visual mesh filename=package://ava_description/meshes/wrist_camera_so101_v1.stl
- added link wrist_camera_frame, mass 1e-9
- added link wrist_camera_mount_link, mass 0.02; collision mesh filename=package://ava_description/meshes/wrist_camera_mount_so101_v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 scale=0.001 0.001 0.001; visual mesh filename=package://ava_description/meshes/wrist_camera_mount_so101_v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 scale=0.001 0.001 0.001
- added link wrist_camera_optical_frame, mass 1e-9
Joints:
- added joint wrist_camera_body_joint: type fixed, parent wrist_camera_mount_link, child wrist_camera_body_link, origin xyz=-0.04941 -0.03813 0.0175 rpy=0 -1.5708 -2.0076
- added joint wrist_camera_frame_joint: type fixed, parent gripper_link, child wrist_camera_frame, origin xyz=0.0025 0.0675 -0.0062 rpy=3.141593 1.136305 -1.570797
- added joint wrist_camera_mount_joint: type fixed, parent gripper_link, child wrist_camera_mount_link, origin xyz=-0.0150 0.0240 -0.0315 rpy=-1.5708 -0.0008 -1.5708
- added joint wrist_camera_optical_joint: type fixed, parent wrist_camera_frame, child wrist_camera_optical_frame, origin xyz=0 0 0 rpy=-1.5708 0 -1.5708

File: ros2_ws/src/ava_description/urdf/ava.urdf.xacro (robot description, xacro)
@@ -42,5 +42,8 @@
   <xacro:arg name="mujoco_headless" default="false"/>
   <!-- false = omit the wrist camera mount/body/frame links and their fixed joints below -->
-  <xacro:arg name="wrist_camera_urdf" default="false"/>
+  <xacro:arg name="wrist_camera_urdf" default="true"/>
+  <!-- Load testing: a point mass at the tool frame (e.g. an object held by the gripper).
+       0 = no payload. Set from gazebo.launch.py payload_kg:=0.1 -->
+  <xacro:arg name="payload_kg" default="0"/>
   <material name="light_grey">
     <color rgba="${light_grey_rgba}"/>
@@ -444,4 +447,21 @@
     <origin xyz="${end_effector_xyz}" rpy="${end_effector_rpy}"/>
   </joint>
+  <xacro:if value="${float('$(arg payload_kg)') > 0}">
+    <link name="payload_link">
+      <inertial>
+        <origin xyz="0 0 0" rpy="0 0 0"/>
+        <mass value="$(arg payload_kg)"/>
+        <inertia ixx="1e-6" iyy="1e-6" izz="1e-6" ixy="0" ixz="0" iyz="0"/>
+      </inertial>
+      <visual>
+        <geometry><sphere radius="0.015"/></geometry>
+        <material name="charcoal"/>
+      </visual>
+    </link>
+    <joint name="payload_joint" type="fixed">
+      <parent link="end_effector_link"/>
+      <child link="payload_link"/>
+    </joint>
+  </xacro:if>
   <xacro:if value="${'$(arg wrist_camera_urdf)' == 'true'}">
     <joint name="wrist_camera_mount_joint" type="fixed">
