Commit message: Replace SO-101 model with in-house CAD design
The SO-101 model failed the Gazebo load test, so the arm was redrawn in
Fusion 360 around a 2x MG996R + 4x SG90 servo budget.

The CAD export is adapted by scripts/generate_kinematics_xacro.py: mesh
paths become package://, collision geometry is kept on the 7 structural
links only, and the six joint limits reference ava.control.xacro. The
export is authored Z-down, so world_to_base rotates pi about X and lifts
the base, or the arm hangs below the ground plane.

SRDF rebuilt. Sampling 600 configurations shows this arm can fold onto
itself, so only the 6 adjacent pairs are disabled where the SO-101 SRDF
disabled 10. Named poses re-verified against the new asymmetric limits.

Joint names are unchanged, so controllers, teleop and the dashboard's
joint plumbing carry over; link names and joint limits do not.

File: ros2_ws/src/ava_description/urdf/ava.common.xacro (robot description, xacro)
@@ -1,33 +1,28 @@
 <?xml version="1.0"?>
+<!-- Shared properties for the Ava arm.
+     Joint origins used to live here; they now come from the CAD export via
+     ava.kinematics.xacro, so only the frames the exporter does not model are left. -->
 <robot xmlns:xacro="http://www.ros.org/wiki/xacro">
   <!-- Color properties (RGBA) -->
   <xacro:property name="light_grey_rgba" value="0.8 0.8 0.8 1.0"/>
   <xacro:property name="charcoal_rgba" value="0.15 0.15 0.15 1.0"/>
-  <!-- Joint origins (from onshape-to-robot calibration) -->
-  <xacro:property name="shoulder_pan_xyz" value="0.0388353 -8.97657e-09 0.0624"/>
-  <xacro:property name="shoulder_lift_xyz" value="0.0303992 -0.0182778 0.0542"/>
-  <xacro:property name="shoulder_lift_rpy" value="-1.5708 1.5708 0"/>
-  <xacro:property name="elbow_flex_xyz" value="-0.11257 -0.028 1.73763e-16"/>
-  <xacro:property name="elbow_flex_rpy" value="-3.63608e-16 8.74301e-16 1.5708"/>
-  <xacro:property name="wrist_flex_xyz" value="-0.1349 0.0052 3.62355e-17"/>
-  <xacro:property name="wrist_flex_rpy" value="4.02456e-15 8.67362e-16 -1.5708"/>
-  <xacro:property name="wrist_roll_xyz" value="5.55112e-17 -0.0611 0.0181"/>
-  <xacro:property name="wrist_roll_rpy" value="1.5708 0.0486795 3.14159"/>
-  <xacro:property name="gripper_xyz" value="0.0202 0.0188 -0.0234"/>
-  <xacro:property name="gripper_rpy" value="1.5708 -5.24284e-08 -1.41553e-15"/>
-  <!-- end_effector_link's rpy (pitch pi/2, not the raw onshape TCP frame) makes its axes X=forward
-       Y=left Z=up like ik_target, instead of the arbitrary CAD TCP orientation. -->
-  <xacro:property name="end_effector_xyz" value="-0.0079 -0.000218121 -0.0981274"/>
-  <xacro:property name="end_effector_rpy" value="0 1.5708 0"/>
-  <!-- SO-101 wrist camera (Hex-Nut Recess mount) reference pose from
-       TheRobotStudio SO-ARM100 + livekit-examples/so-frame. -->
-  <xacro:property name="wrist_camera_mount_xyz" value="-0.0150 0.0240 -0.0315"/>
-  <xacro:property name="wrist_camera_mount_rpy" value="-1.5708 -0.0008 -1.5708"/>
-  <!-- Camera body mesh pose and scale relative to wrist_camera_mount_link. -->
-  <xacro:property name="wrist_camera_body_xyz" value="-0.04941 -0.03813 0.0175"/>
-  <xacro:property name="wrist_camera_body_rpy" value="0 -1.5708 -2.0076"/>
-  <!-- Non-REP-103 camera frame that follows upstream so-frame alignment. -->
-  <xacro:property name="wrist_camera_frame_xyz" value="0.0025 0.0675 -0.0062"/>
-  <xacro:property name="wrist_camera_frame_rpy" value="3.141593 1.136305 -1.570797"/>
+  <!-- Height of base_link's underside above base_footprint, after the Z-down export is
+       flipped pi about X (see world_to_base in ava.urdf.xacro). Measured from the
+       base_link collision mesh: it spans z=-0.0843..+0.0337 once flipped. -->
+  <xacro:property name="base_mount_z" value="0.0337"/>
+  <!-- Tool frame, in the gripper_base_link frame. Measured from the gripper meshes:
+       the jaws span x=-0.0676..-0.002 and the body reaches x=-0.0705, so the grasp point
+       sits just inside the jaw tips. end_effector_link's rpy yaws pi so its axes read
+       X=approach Y=left Z=up like ik_target, instead of the CAD part orientation. -->
+  <xacro:property name="end_effector_xyz" value="-0.065 0.003 -0.025"/>
+  <xacro:property name="end_effector_rpy" value="0 0 3.141593"/>
+  <!-- Wrist camera: PLACEHOLDER extrinsics. The redesign has no camera mount part, so
+       there is nothing in the CAD model to measure these against. The frames exist only
+       so ava_vision's TF lookups resolve; re-measure on hardware before relying on them.
+       See the wrist_camera_urdf arg in ava.urdf.xacro to omit them entirely. -->
+  <xacro:property name="wrist_camera_mount_xyz" value="0 0 0"/>
+  <xacro:property name="wrist_camera_mount_rpy" value="0 0 0"/>
+  <xacro:property name="wrist_camera_frame_xyz" value="0 0 0"/>
+  <xacro:property name="wrist_camera_frame_rpy" value="0 0 0"/>
   <!-- REP-103 optical frame (+Z forward, +X right, +Y down) as child of wrist_camera_frame. -->
   <xacro:property name="wrist_camera_optical_rpy" value="-1.5708 0 -1.5708"/>

File: ros2_ws/src/ava_description/urdf/ava.control.xacro (robot description, xacro)
@@ -43,16 +43,31 @@
   <!-- Position insensitive-area (CW_DEAD/CCW_DEAD, both set to this value) -->
   <xacro:property name="deadband" value="10"/>
-  <!-- Joint limits (from onshape-to-robot calibration) -->
-  <xacro:property name="shoulder_pan_lower" value="-1.91986"/>
-  <xacro:property name="shoulder_pan_upper" value="1.91986"/>
-  <xacro:property name="shoulder_lift_lower" value="-1.74533"/>
-  <xacro:property name="shoulder_lift_upper" value="1.74533"/>
-  <xacro:property name="elbow_flex_lower" value="-1.69"/>
-  <xacro:property name="elbow_flex_upper" value="1.69"/>
-  <xacro:property name="wrist_flex_lower" value="-1.65806"/>
-  <xacro:property name="wrist_flex_upper" value="1.65806"/>
-  <xacro:property name="wrist_roll_lower" value="-2.74385"/>
-  <xacro:property name="wrist_roll_upper" value="2.84121"/>
-  <xacro:property name="gripper_lower" value="-1.74533"/>
-  <xacro:property name="gripper_upper" value="0.174533"/>
+  <!-- Joint limits and per-joint effort ceilings.
+       GENERATED VALUES: these mirror the <limit> tags of the current CAD export
+       (urdf/ava_robotic_arm.urdf). ava.kinematics.xacro references them by name so the
+       numbers stay reviewable here rather than buried in the 45-link export. If you
+       re-export the model with changed limits, update these to match. -->
+  <xacro:property name="shoulder_pan_lower" value="-1.570796"/>
+  <xacro:property name="shoulder_pan_upper" value="1.570796"/>
+  <xacro:property name="shoulder_lift_lower" value="-0.212536"/>
+  <xacro:property name="shoulder_lift_upper" value="2.094395"/>
+  <xacro:property name="elbow_flex_lower" value="-1.523672"/>
+  <xacro:property name="elbow_flex_upper" value="1.617920"/>
+  <xacro:property name="wrist_flex_lower" value="-2.617994"/>
+  <xacro:property name="wrist_flex_upper" value="0.523599"/>
+  <xacro:property name="wrist_roll_lower" value="-1.963495"/>
+  <xacro:property name="wrist_roll_upper" value="1.178097"/>
+  <xacro:property name="gripper_lower" value="-0.594434"/>
+  <xacro:property name="gripper_upper" value="0.197952"/>
+  <!-- Per-joint effort ceilings (N*m). The redesign is no longer a uniform STS3215 bus:
+       the CAD model is built around MG996R servos at the shoulder and SG90s from the
+       elbow out, so effort now differs per joint instead of sharing max_torque_nm.
+       NOTE: ava.ros2control.xacro still drives this arm as an STS3215 serial bus
+       (motor IDs, EEPROM PID writes). That hardware layer has not been retargeted. -->
+  <xacro:property name="shoulder_pan_effort" value="1.079"/>   <!-- MG996R -->
+  <xacro:property name="shoulder_lift_effort" value="2.157"/>  <!-- MG996R, geared -->
+  <xacro:property name="elbow_flex_effort" value="0.177"/>     <!-- SG90 -->
+  <xacro:property name="wrist_flex_effort" value="0.177"/>      <!-- SG90 -->
+  <xacro:property name="wrist_roll_effort" value="0.177"/>      <!-- SG90 -->
+  <xacro:property name="gripper_effort" value="0.177"/>         <!-- SG90 -->
 </robot>
