Commit message: Elbow to MG996R, real servo ratings, Gazebo load-test results
3x MG996R + 3x SG90 layout; SG90 1.6 kg*cm
and MG996R 11 kg*cm at 6 V; no geared shoulder.
Gazebo sweep: holds 20 g payload, wrist_flex fails
at 50 g (docs/simulation_validation.md).
Removed broken OmArm hardware bridges and STS3215
params; ava_hardware plugin parked (COLCON_IGNORE).
New docs: robot spec, decisions, simulation testing
guide, validation templates.
Fusion design still under construction (elbow mount
being redrawn).

File: ros2_ws/src/ava_description/urdf/ava.urdf.xacro (robot description, xacro)
@@ -3,39 +3,12 @@
   <xacro:include filename="$(find ava_description)/urdf/ava.common.xacro"/>
   <xacro:include filename="$(find ava_description)/urdf/ava.control.xacro"/>
-  <!-- Arguments (externally settable, default to property values in ava.control.xacro) -->
-  <xacro:arg name="serial_port"    default="${serial_port}"/>
-  <xacro:arg name="baud_rate"      default="${baud_rate}"/>
-  <xacro:arg name="use_mock"       default="${use_mock}"/>
-  <xacro:arg name="use_sync_write" default="${use_sync_write}"/>
-  <xacro:arg name="arm_operating_mode"     default="${arm_operating_mode}"/>     <!-- 0=Position 1=Velocity 2=PWM; arm joints 1-5; baked at startup -->
-  <xacro:arg name="gripper_operating_mode" default="${gripper_operating_mode}"/> <!-- 0=Position 1=Velocity 2=PWM; gripper joint 6; baked at startup -->
-  <xacro:arg name="shoulder_pan_motor_id" default="${shoulder_pan_motor_id}"/>
-  <xacro:arg name="shoulder_lift_motor_id" default="${shoulder_lift_motor_id}"/>
-  <xacro:arg name="elbow_flex_motor_id" default="${elbow_flex_motor_id}"/>
-  <xacro:arg name="wrist_flex_motor_id" default="${wrist_flex_motor_id}"/>
-  <xacro:arg name="wrist_roll_motor_id" default="${wrist_roll_motor_id}"/>
-  <xacro:arg name="gripper_motor_id" default="${gripper_motor_id}"/>
-  <xacro:arg name="shoulder_pan_p_coefficient" default="${shoulder_pan_p_coefficient}"/>
-  <xacro:arg name="shoulder_pan_d_coefficient" default="${shoulder_pan_d_coefficient}"/>
-  <xacro:arg name="shoulder_pan_i_coefficient" default="${shoulder_pan_i_coefficient}"/>
-  <xacro:arg name="shoulder_lift_p_coefficient" default="${shoulder_lift_p_coefficient}"/>
-  <xacro:arg name="shoulder_lift_d_coefficient" default="${shoulder_lift_d_coefficient}"/>
-  <xacro:arg name="shoulder_lift_i_coefficient" default="${shoulder_lift_i_coefficient}"/>
-  <xacro:arg name="elbow_flex_p_coefficient" default="${elbow_flex_p_coefficient}"/>
-  <xacro:arg name="elbow_flex_d_coefficient" default="${elbow_flex_d_coefficient}"/>
-  <xacro:arg name="elbow_flex_i_coefficient" default="${elbow_flex_i_coefficient}"/>
-  <xacro:arg name="wrist_flex_p_coefficient" default="${wrist_flex_p_coefficient}"/>
-  <xacro:arg name="wrist_flex_d_coefficient" default="${wrist_flex_d_coefficient}"/>
-  <xacro:arg name="wrist_flex_i_coefficient" default="${wrist_flex_i_coefficient}"/>
-  <xacro:arg name="wrist_roll_p_coefficient" default="${wrist_roll_p_coefficient}"/>
-  <xacro:arg name="wrist_roll_d_coefficient" default="${wrist_roll_d_coefficient}"/>
-  <xacro:arg name="wrist_roll_i_coefficient" default="${wrist_roll_i_coefficient}"/>
-  <xacro:arg name="gripper_p_coefficient" default="${gripper_p_coefficient}"/>
-  <xacro:arg name="gripper_d_coefficient" default="${gripper_d_coefficient}"/>
-  <xacro:arg name="gripper_i_coefficient" default="${gripper_i_coefficient}"/>
-  <xacro:arg name="deadband" default="${deadband}"/>
-  <!-- real=STS serial plugin, gazebo=gz_ros2_control, mujoco=MujocoSystemInterface,
-       mock_components=GenericSystem. Selects the <hardware> block in ava.ros2control.xacro. -->
-  <xacro:arg name="ros2_control_hardware_type" default="real"/>
+  <!-- Real hardware only: USB serial port of the ESP32 servo driver and its baud rate. -->
+  <xacro:arg name="serial_port" default="/dev/ttyUSB0"/>
+  <xacro:arg name="baud_rate"   default="115200"/>
+  <!-- Selects the <hardware> block in ava.ros2control.xacro:
+       real=ava_hardware/AvaServoSystem (ESP32 + PCA9685 PWM servos over USB serial),
+       gazebo=gz_ros2_control, mujoco=MujocoSystemInterface, mock_components=GenericSystem.
+       Defaults to mock_components so a bare xacro call never talks to hardware. -->
+  <xacro:arg name="ros2_control_hardware_type" default="mock_components"/>
   <!-- mujoco only -->
   <xacro:arg name="mujoco_model" default=""/>
@@ -98,4 +71,22 @@
     </joint>
   </xacro:if>
+  <!-- TEMPORARY until the redrawn CAD export arrives: the elbow is now an MG996R, but the
+       current export still carries an SG90 body (sg90R_01, 9.5 g) on the upper arm. This
+       point mass adds the difference (MG996R body 56.3 g - SG90 body 9.5 g = 46.8 g) at that
+       SG90's centre of mass, so Gazebo loads the shoulder with the heavier servo. Position is
+       sg90R_01's CoM expressed in upper_arm_link; inertia is a rough 40x19x43 mm box.
+       Delete this block when the new export (with an MG996R at the elbow) is dropped in. -->
+  <link name="elbow_servo_mass_stub">
+    <inertial>
+      <origin xyz="0 0 0" rpy="0 0 0"/>
+      <mass value="0.0468"/>
+      <inertia ixx="1e-5" iyy="1e-5" izz="1e-5" ixy="0" ixz="0" iyz="0"/>
+    </inertial>
+  </link>
+  <joint name="elbow_servo_mass_stub_joint" type="fixed">
+    <parent link="upper_arm_link"/>
+    <child link="elbow_servo_mass_stub"/>
+    <origin xyz="0.0473 -0.0147 -0.1370" rpy="0 0 0"/>
+  </joint>
   <!-- WRIST CAMERA: frames only. The redesign has no camera mount part, so the SO-101
        mount and camera-body meshes are gone and these poses are PLACEHOLDERS - the frames

Commit message: feat(hardware): ava_hardware, rest pose, smooth park, wiring docs

File: ros2_ws/src/ava_description/urdf/ava.control.xacro (robot description, xacro)
@@ -14,8 +14,10 @@
   <xacro:property name="servo_max_us" value="2500"/>
   <!-- Serial link to the ESP32. The ESP32 resets when the port is opened, so the handshake
-       waits for it to boot. release_on_deactivate=true sends "D" (all servos limp) when the
-       hardware is deactivated; false keeps the last pulses held. -->
+       waits for it to boot. On deactivation (Ctrl+C) the arm first moves smoothly to its rest
+       pose in servo_park_duration_s (0 = no parking, max 4); then release_on_deactivate=true
+       sends "D" (all servos limp), false keeps the rest pose held. -->
   <xacro:property name="servo_handshake_timeout_ms" value="4000"/>
   <xacro:property name="servo_release_on_deactivate" value="false"/>
+  <xacro:property name="servo_park_duration_s" value="2.0"/>
   <!-- PCA9685 channel per joint (J-number = channel + 1). -->
   <xacro:property name="shoulder_pan_channel" value="0"/>   <!-- J1 MG996R -->
@@ -51,4 +53,13 @@
   <xacro:property name="wrist_roll_max_velocity" value="8.73"/>     <!-- SG90 -->
   <xacro:property name="gripper_max_velocity" value="8.73"/>        <!-- SG90 -->
+  <!-- Rest pose (rad): the arm goes here on activation and parks here before shutdown. Set it to
+       the pose the assembled arm sits in when unpowered, so start-up barely moves it. Must lie
+       inside the joint limits below. 0 = the SRDF "home" pose. -->
+  <xacro:property name="shoulder_pan_rest" value="0.0"/>
+  <xacro:property name="shoulder_lift_rest" value="0.0"/>
+  <xacro:property name="elbow_flex_rest" value="0.0"/>
+  <xacro:property name="wrist_flex_rest" value="0.0"/>
+  <xacro:property name="wrist_roll_rest" value="0.0"/>
+  <xacro:property name="gripper_rest" value="0.0"/>
   <!-- Joint limits.
        GENERATED VALUES: these mirror the <limit> tags of the current CAD export

File: ros2_ws/src/ava_description/urdf/ava.ros2control.xacro (robot description, xacro)
@@ -13,5 +13,5 @@
        q = 0) is derived from the pulse at mid-range:
          zero_us = center_us - direction * (lower + upper) / 2 * servo_us_per_rad -->
-  <xacro:macro name="ava_servo_joint" params="name channel direction center_us max_velocity lower upper">
+  <xacro:macro name="ava_servo_joint" params="name channel direction center_us max_velocity lower upper rest">
     <joint name="${name}">
       <xacro:if value="${hw_type == 'real'}">
@@ -25,4 +25,5 @@
         <param name="min_position">${lower}</param>
         <param name="max_position">${upper}</param>
+        <param name="rest_position">${rest}</param>
       </xacro:if>
       <command_interface name="position"/>
@@ -48,6 +49,6 @@
         <plugin>mock_components/GenericSystem</plugin>
       </xacro:if>
-      <!-- ESP32 + PCA9685 over USB serial (package ava_hardware). NOTE: activation commands
-           every joint to 0 rad, so the arm jumps to the home pose at start-up. -->
+      <!-- ESP32 + PCA9685 over USB serial (package ava_hardware). Activation commands the rest
+           pose (ava.control.xacro); deactivation parks the arm there first. -->
       <xacro:if value="${hw_type == 'real'}">
         <plugin>ava_hardware/AvaServoSystem</plugin>
@@ -56,4 +57,5 @@
         <param name="handshake_timeout_ms">${servo_handshake_timeout_ms}</param>
         <param name="release_on_deactivate">${str(servo_release_on_deactivate).lower()}</param>
+        <param name="park_duration_s">${servo_park_duration_s}</param>
       </xacro:if>
     </hardware>
@@ -61,25 +63,25 @@
       direction="${shoulder_pan_direction}" center_us="${shoulder_pan_center_us}"
       max_velocity="${shoulder_pan_max_velocity}"
-      lower="${shoulder_pan_lower}" upper="${shoulder_pan_upper}"/>
+      lower="${shoulder_pan_lower}" upper="${shoulder_pan_upper}" rest="${shoulder_pan_rest}"/>
     <xacro:ava_servo_joint name="shoulder_lift" channel="${shoulder_lift_channel}"
       direction="${shoulder_lift_direction}" center_us="${shoulder_lift_center_us}"
       max_velocity="${shoulder_lift_max_velocity}"
-      lower="${shoulder_lift_lower}" upper="${shoulder_lift_upper}"/>
+      lower="${shoulder_lift_lower}" upper="${shoulder_lift_upper}" rest="${shoulder_lift_rest}"/>
     <xacro:ava_servo_joint name="elbow_flex" channel="${elbow_flex_channel}"
       direction="${elbow_flex_direction}" center_us="${elbow_flex_center_us}"
       max_velocity="${elbow_flex_max_velocity}"
-      lower="${elbow_flex_lower}" upper="${elbow_flex_upper}"/>
+      lower="${elbow_flex_lower}" upper="${elbow_flex_upper}" rest="${elbow_flex_rest}"/>
     <xacro:ava_servo_joint name="wrist_flex" channel="${wrist_flex_channel}"
       direction="${wrist_flex_direction}" center_us="${wrist_flex_center_us}"
       max_velocity="${wrist_flex_max_velocity}"
-      lower="${wrist_flex_lower}" upper="${wrist_flex_upper}"/>
+      lower="${wrist_flex_lower}" upper="${wrist_flex_upper}" rest="${wrist_flex_rest}"/>
     <xacro:ava_servo_joint name="wrist_roll" channel="${wrist_roll_channel}"
       direction="${wrist_roll_direction}" center_us="${wrist_roll_center_us}"
       max_velocity="${wrist_roll_max_velocity}"
-      lower="${wrist_roll_lower}" upper="${wrist_roll_upper}"/>
+      lower="${wrist_roll_lower}" upper="${wrist_roll_upper}" rest="${wrist_roll_rest}"/>
     <xacro:ava_servo_joint name="gripper" channel="${gripper_channel}"
       direction="${gripper_direction}" center_us="${gripper_center_us}"
       max_velocity="${gripper_max_velocity}"
-      lower="${gripper_lower}" upper="${gripper_upper}"/>
+      lower="${gripper_lower}" upper="${gripper_upper}" rest="${gripper_rest}"/>
   </ros2_control>
 </robot>
